File: kicad/card.kicad_pcb (KiCad board)
At the start: 2 copper layers, 83.1 x 91.2 mm, 80 parts, among them J1 USB_B_Mini, J10 Conn_01x04, J11 Conn_01x08, J12 Conn_01x04, J13 Conn_02x03_Odd_Even, J14 Conn_01x02, J15 3V3, J16 3V3, J17 Conn_01x08, J18 3V3, J19 Conn_01x02, J2 Conn_02x03_Odd_Even, J20 3V3, J21 Conn_01x01_Male, J3 Conn_01x04, J4 Conn_01x02, J5 Conn_01x04, J6 Conn_01x02, J7 Conn_01x02, J8 Conn_01x07_RGB, J9 Conn_01x03, Q1 BSS138, U1 ATmega32U2-AU, U2 EPM3064_KbdHub, U3 MAX3421EEHJ+T, U4 IP4220CZ6, U5 EPM3032, U6 AP7215-33YG-13, U7 ExtHub, U8 AP7215-33YG-13, X1 ScorpionEdgeConnector, X2 ScorpionBusConnector, Y1 12M, Y2 16M

Commit message: Sources updated
Parts:
- R5: value 1K -> 1K2
- R6: value 1K -> 0
Connections:
- J21 pad 1: ZRES -> Net-(J21-Pad1)
- R9 pad 1: ZRES_E -> ZRES
- R9 pad 2: ZRES -> Net-(J21-Pad1)
- U1 pad 9: ZRES -> Net-(J21-Pad1)
- U5 pad 21: (no net) -> MC_RES
- X1 pad 19: ZRES_E -> ZRES
Routing:
- net ZRES_E: track 12.3 -> 0.00 mm
- net Net-(J21-Pad1): track 0.00 -> 9.86 mm
- net MC_RES: track 48.2 -> 57.1 mm, vias 2 -> 4
- net GND: track 239.6 -> 247.7 mm
- net ZRES: track 9.86 -> 12.3 mm
Other:
- board text added: "revA2"
