File: kicad/card.kicad_sch (KiCad schematic)
At the start: 80 parts, among them J1 USB_B_Mini, J10 Conn_01x04, J11 Conn_01x08, J12 Conn_01x04, J13 Conn_02x03_Odd_Even, J14 Conn_01x02, J15 3V3, J16 3V3, J17 Conn_01x08, J18 3V3, J19 Conn_01x02, J2 Conn_02x03_Odd_Even, J20 3V3, J21 Conn_01x01_Male, J3 Conn_01x04, J4 Conn_01x02, J5 Conn_01x04, J6 Conn_01x02, J7 Conn_01x02, J8 Conn_01x07_RGB, J9 Conn_01x03, Q1 BSS138, U1 ATmega32U2-AU, U2 EPM3064_KbdHub, U3 MAX3421EEHJ+T, U4 IP4220CZ6, U5 EPM3032, U6 AP7215-33YG-13, U7 ExtHub, U8 AP7215-33YG-13, X1 ScorpionEdgeConnector, X2 ScorpionBusConnector, Y1 12M, Y2 16M

Commit message: Sources updated
Parts:
- C3: value (none) -> 1µF; footprint (none) -> Capacitor_SMD:C_0805_2012Metric
- R5: value 1K -> 1K2
- R6: value 1K -> 0
Connections:
- net ZRES_E is gone; now on net ZRES: R9.1, X1.19 (RESET)
- net MC_RES: now also U5.21 (RST)
- net ZRES: no longer J21.1 (Pin_1), R9.2, U1.9 (PD3)
- new net: J21.1 (Pin_1), R9.2, U1.9 (PD3)
Other:
- moved on the sheet: J21, R9
Changed lines of the file:
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@@
 (kicad_sch (version 20211123) (generator eeschema)
   (paper "A4")
-  (junction (at 266.7 83.82) (diameter 0) (color 0 0 0 0)
-  )
   (junction (at 246.38 88.9) (diameter 0) (color 0 0 0 0)
   )
@@
   (junction (at 241.3 96.52) (diameter 0) (color 0 0 0 0)
   )
+  (junction (at 99.06 68.58) (diameter 0) (color 0 0 0 0)
+  )
   (junction (at 280.67 109.22) (diameter 0) (color 0 0 0 0)
   )
@@
     (stroke (width 0) (type default) (color 0 0 0 0))
   )
+  (wire (pts (xy 99.06 68.58) (xy 99.06 71.12))
+    (stroke (width 0) (type default) (color 0 0 0 0))
+  )
   (wire (pts (xy 251.46 96.52) (xy 256.54 96.52))
     (stroke (width 0) (type default) (color 0 0 0 0))
@@
     (stroke (width 0) (type default) (color 0 0 0 0))
   )
+  (wire (pts (xy 93.98 68.58) (xy 99.06 68.58))
+    (stroke (width 0) (type default) (color 0 0 0 0))
+  )
   (wire (pts (xy 278.13 22.86) (xy 278.13 27.94))
     (stroke (width 0) (type default) (color 0 0 0 0))
@@
     (stroke (width 0) (type default) (color 0 0 0 0))
   )
+  (wire (pts (xy 99.06 71.12) (xy 104.14 71.12))
+    (stroke (width 0) (type default) (color 0 0 0 0))
+  )
   (wire (pts (xy 149.86 139.7) (xy 147.32 139.7))
     (stroke (width 0) (type default) (color 0 0 0 0))
@@
     (stroke (width 0) (type default) (color 0 0 0 0))
   )
-  (wire (pts (xy 266.7 80.01) (xy 271.78 80.01))
-    (stroke (width 0) (type default) (color 0 0 0 0))
-  )
   (wire (pts (xy 186.69 15.24) (xy 186.69 31.75))
     (stroke (width 0) (type default) (color 0 0 0 0))
@@
     (stroke (width 0) (type default) (color 0 0 0 0))
   )
-  (wire (pts (xy 266.7 83.82) (xy 266.7 80.01))
-    (stroke (width 0) (type default) (color 0 0 0 0))
-  )
   (wire (pts (xy 271.78 88.9) (xy 276.86 88.9))
     (stroke (width 0) (type default) (color 0 0 0 0))
@@
     )
   )
-  (global_label "ZRES_E" (shape input) (at 22.86 135.89 180) (fields_autoplaced)
+  (global_label "ZRES" (shape input) (at 22.86 135.89 180) (fields_autoplaced)
     (effects (font (size 1.27 1.27)) (justify right))
-    (property "Intersheet References" "${INTERSHEET_REFS}" (id 0) (at 13.581 135.8106 0)
+    (property "Intersheet References" "${INTERSHEET_REFS}" (id 0) (at 15.6977 135.8106 0)
       (effects (font (size 1.27 1.27)) (justify right) hide)
     )
@@
     )
   )
-  (global_label "ZRES_E" (shape input) (at 271.78 83.82 0) (fields_autoplaced)
+  (global_label "ZRES" (shape input) (at 104.14 68.58 0) (fields_autoplaced)
     (effects (font (size 1.27 1.27)) (justify left))
-    (property "Intersheet References" "${INTERSHEET_REFS}" (id 0) (at 281.059 83.7406 0)
+    (property "Intersheet References" "${INTERSHEET_REFS}" (id 0) (at 111.3023 68.5006 0)
       (effects (font (size 1.27 1.27)) (justify left) hide)
     )
@@
     )
   )
-  (global_label "ZRES" (shape input) (at 93.98 68.58 0) (fields_autoplaced)
-    (effects (font (size 1.27 1.27)) (justify left))
-    (property "Intersheet References" "${INTERSHEET_REFS}" (id 0) (at 0 2.54 0)
-      (effects (font (size 1.27 1.27)) hide)
-    )
-  )
   (global_label "MC_RES" (shape input) (at 58.42 22.86 180) (fields_autoplaced)
     (effects (font (size 1.27 1.27)) (justify right))
@@
     )
   )
-  (global_label "ZRES" (shape input) (at 271.78 80.01 0) (fields_autoplaced)
-    (effects (font (size 1.27 1.27)) (justify left))
-    (property "Intersheet References" "${INTERSHEET_REFS}" (id 0) (at 278.9423 79.9306 0)
-      (effects (font (size 1.27 1.27)) (justify left) hide)
-    )
-  )
   (global_label "A1" (shape input) (at 99.06 135.89 180) (fields_autoplaced)
     (effects (font (size 1.27 1.27)) (justify right))
@@
     )
   )
+  (global_label "MC_RES" (shape input) (at 201.93 68.58 180) (fields_autoplaced)
+    (effects (font (size 1.27 1.27)) (justify right))
+    (property "Intersheet References" "${INTERSHEET_REFS}" (id 0) (at 192.2882 68.5006 0)
+      (effects (font (size 1.27 1.27)) (justify right) hide)
+    )
+  )
   (global_label "EINT" (shape input) (at 93.98 55.88 0) (fields_autoplaced)
     (effects (font (size 1.27 1.27)) (justify left))
@@
       (effects (font (size 1.27 1.27)) (justify left))
     )
-    (property "Value" "" (id 1) (at 53.34 53.34 0)
+    (property "Value" "1µF" (id 1) (at 53.34 53.34 0)
       (effects (font (size 1.27 1.27)) (justify left))
     )
-    (property "Footprint" "" (id 2) (at 58.1152 54.61 0)
+    (property "Footprint" "Capacitor_SMD:C_0805_2012Metric" (id 2) (at 58.1152 54.61 0)
       (effects (font (size 1.27 1.27)) hide)
     )
@@
       (effects (font (size 1.27 1.27)) (justify left))
     )
-    (property "Value" "1K" (id 1) (at 104.14 86.36 90)
+    (property "Value" "0" (id 1) (at 104.14 86.36 90)
       (effects (font (size 1.27 1.27)) (justify left))
     )
@@
     (pin "37")
     (pin "38")
+    (pin "21")
     (pin "39")
     (pin "4")
@@
   (symbol (lib_id "Device:C") (at 121.92 87.63 0) (unit 1)
     (in_bom yes) (on_board yes)
-    (property "Reference" "C4" (id 0) (at 119.38 85.09 0)
+    (property "Reference" "C4" (id 0) (at 121.92 90.17 0)
       (effects (font (size 1.27 1.27)) (justify left))
     )
-    (property "Value" "10nF" (id 1) (at 119.38 90.17 0)
+    (property "Value" "10nF" (id 1) (at 123.19 86.36 90)
       (effects (font (size 1.27 1.27)) (justify left))
     )
@@
       (effects (font (size 1.27 1.27)) (justify left))
     )
-    (property "Value" "1K" (id 1) (at 123.698 78.613 0)
+    (property "Value" "1K2" (id 1) (at 123.698 78.613 0)
       (effects (font (size 1.27 1.27)) (justify left))
     )
@@
     (pin "2")
   )
-  (symbol (lib_id "Device:R_Small") (at 269.24 83.82 270) (unit 1)
+  (symbol (lib_id "Device:R_Small") (at 101.6 68.58 270) (unit 1)
     (in_bom yes) (on_board yes)
-    (property "Reference" "R9" (id 0) (at 269.24 83.82 90))
-    (property "Value" "250" (id 1) (at 269.24 81.28 90))
-    (property "Footprint" "Resistor_SMD:R_0805_2012Metric" (id 2) (at 269.24 83.82 0)
+    (property "Reference" "R9" (id 0) (at 101.6 68.58 90))
+    (property "Value" "250" (id 1) (at 101.6 66.04 90))
+    (property "Footprint" "Resistor_SMD:R_0805_2012Metric" (id 2) (at 101.6 68.58 0)
       (effects (font (size 1.27 1.27)) hide)
     )
-    (property "Datasheet" "~" (id 3) (at 269.24 83.82 0)
+    (property "Datasheet" "~" (id 3) (at 101.6 68.58 0)
       (effects (font (size 1.27 1.27)) hide)
     )
@@
     (pin "1")
   )
-  (symbol (lib_id "Connector:Conn_01x01_Male") (at 261.62 83.82 0) (unit 1)
+  (symbol (lib_id "Connector:Conn_01x01_Male") (at 109.22 71.12 180) (unit 1)
     (in_bom yes) (on_board yes)
-    (property "Reference" "J21" (id 0) (at 264.16 85.09 0))
-    (property "Value" "Conn_01x01_Male" (id 1) (at 262.255 81.28 0)
+    (property "Reference" "J21" (id 0) (at 111.76 71.12 0))
+    (property "Value" "Conn_01x01_Male" (id 1) (at 108.585 73.66 0)
       (effects (font (size 1.27 1.27)) hide)
     )
-    (property "Footprint" "Connector_PinHeader_2.54mm:PinHeader_1x01_P2.54mm_Vertical" (id 2) (at 261.62 83.82 0)
+    (property "Footprint" "Connector_PinHeader_2.54mm:PinHeader_1x01_P2.54mm_Vertical" (id 2) (at 109.22 71.12 0)
       (effects (font (size 1.27 1.27)) hide)
     )
-    (property "Datasheet" "~" (id 3) (at 261.62 83.82 0)
+    (property "Datasheet" "~" (id 3) (at 109.22 71.12 0)
       (effects (font (size 1.27 1.27)) hide)
     )
@@
     )
     (path "/00000000-0000-0000-0000-00006283bf59"
-      (reference "R5") (unit 1) (value "1K") (footprint "Resistor_SMD:R_0805_2012Metric")
+      (reference "R5") (unit 1) (value "1K2") (footprint "Resistor_SMD:R_0805_2012Metric")
     )
     (path "/00000000-0000-0000-0000-0000626460b4"
-      (reference "R6") (unit 1) (value "1K") (footprint "Resistor_SMD:R_0805_2012Metric")
+      (reference "R6") (unit 1) (value "0") (footprint "Resistor_SMD:R_0805_2012Metric")
     )
     (path "/00000000-0000-0000-0000-000062552687"
